File: Alta.sch (EAGLE design)
At the start: 13 parts

Commit message: Rev4 - Adição do circuito de Alta Latência - Previsão de conexão de módulos de expansão - Correção de falhas e previsão de melhorias com relação a estabilidade do sistema - Definição dos valores iniciais para cada componente - Previsão de circuito conversor de nivel para possivel feature implementável de atualização de firmware.
Parts:
- removed C31: 2200uf/35V, rcl:CPOL-EUE3.5-10
- removed F1: 5A/250V, fuse:KS9V
- removed JP74, JP76, JP77, JP78, JP79, JP80, JP81, JP82: (no value), jumper:JP1E
- removed LED1: (no value), led:LED3MM
- removed R44: 4 m, resistor-shunt:PMA-B
- removed R49: 470, rcl:R-US_0613/5V
- added C1, C2: 100nf/50V, rcl:C-EUC0603K
- added C10, C11, C12, C13, C14, C15, C19, C20, C21, C22, C23, C24, C25: 1nf/50V, rcl:C-EUC0603K
- added C16, C17, C18, C3, C9: 10nf/50V, rcl:C-EUC0603K
- added C6: 470uf/35V, rcl:CPOL-EU140CLH-1014
- added C7, C8: 100nf/50V, rcl:C-EUC0805
- added D1: S1J, diode:DIODE-SMC
- added D2: BAS21, diode:BAS40
- added JP11: (no value), jumper:JP1Q
- added L1: 330m, inductor-neosid:MS50
- added LSP1, LSP2, LSP3: LSP10, solpad:LSP10
- added Q1, Q5, Q6, Q7: BC817, transistor-npn:BC817-16LT1SMD
- added Q2, Q3, Q4: BC807, transistor-pnp:BC807-40SMD
- added R1, R24, R25, R26: 150k, rcl:R-EU_R0603
- added R10, R11, R12, R13, R14, R2, R27, R28, R29, R9: 100k, rcl:R-EU_R0603
- added R15, R16, R17, R18, R19, R20, R37, R38, R39, R40, R41, R42, R43: 100, rcl:R-EU_R0603
- added R21, R22, R23, R3, R30, R31, R32, R33, R34, R35, R36, R4, R5, R6, R7, R8: 10k, rcl:R-EU_R0603
- added S1, S10, S11, S12, S13, S2, S3, S4, S5, S6, S7, S8, S9: (no value), SparkFun-Electromechanical:TAC_SWITCHSMD
- added SG1: F/CM12P, buzzer:F/CM12P
- added X1: RASPBERRYPI-B+-GPIO, SparkFun-Boards:RASPBERRYPI-B+-GPIO
- added Z1: 5v1, diode:BAS70
Connections:
- removed net N$170: LED1.A, R49.1
- removed net N$171: F1.2, R44.B
- removed net N$172: F1.1, JP74.1, JP74.2, JP76.1, JP76.2, JP77.1, JP77.2
- removed net SHUNT_1: R44.SB
- removed net SHUNT_2: R44.SA
- new net +3V3: C1.1, C2.1, R3.2, R30.2, R31.2, R32.2, R33.2, R34.2, R35.2, R36.2, R4.2, R5.2, R6.2, R7.2, R8.2, X1.3.3V@1, X1.3.3V@17
- new net B01: C15.1, R8.1, S6.3, S6.4, X1.GP5
- new net B02: C14.1, R7.1, S5.3, S5.4, X1.GP6
- new net B03: C13.1, R6.1, S4.3, S4.4, X1.GP12
- new net B04: C12.1, R5.1, S3.3, S3.4, X1.GP13
- new net B05: C11.1, R4.1, S2.3, S2.4, X1.GP16
- new net B06: C10.1, R3.1, S1.3, S1.4, X1.GP19
- new net BACKSPACE: C24.1, R35.1, S12.3, S12.4, X1.GP27
- new net BUZZER: R1.1, X1.GP22
- new net DOWN: C19.1, R30.1, S7.3, S7.4, X1.GP24
- new net ENTER: C25.1, R36.1, S13.3, S13.4, X1.GP26
- new net ESC: C23.1, R34.1, S11.3, S11.4, X1.GP20
- new net ESPAÇO: C22.1, R33.1, S10.3, S10.4, X1.GP21
- new net FIM: C21.1, R32.1, S9.3, S9.4, X1.GP23
- new net MCLR: R24.1, X1.GP18#
- new net N$100: X1.SCLK
- new net N$101: X1.RXI
- new net N$102: X1.TXO
- new net N$103: X1.SCL
- new net N$104: X1.SDA
- new net N$105: Q7.C, R14.1
- new net N$106: C18.1, Q7.B, R26.2, R29.2
- new net N$107: Q4.B, R11.1, R14.2
- new net N$108: LSP3.MP, Q4.C, R23.2
- new net N$117: Q6.C, R13.1
- new net N$119: C17.1, Q6.B, R25.2, R28.2
- new net N$120: Q3.B, R10.1, R13.2
- new net N$121: LSP2.MP, Q3.C, R22.2
- new net N$122: Q5.C, R12.1
- new net N$123: C16.1, Q5.B, R24.2, R27.2
- new net N$124: Q2.B, R12.2, R9.1
- new net N$125: LSP1.MP, Q2.C, R21.2
- new net N$76: D1.A, JP11.2
- new net N$77: C6.+, C7.1, C8.1, D1.C, L1.1, Z1.C
- new net N$78: R20.2, S6.1, S6.2
- new net N$79: R15.2, S1.1, S1.2
- new net N$80: R16.2, S2.1, S2.2
- new net N$81: R17.2, S3.1, S3.2
- new net N$82: R18.2, S4.1, S4.2
- new net N$83: R19.2, S5.1, S5.2
- new net N$84: R43.2, S13.1, S13.2
- new net N$86: R38.2, S8.1, S8.2
- new net N$87: R39.2, S9.1, S9.2
- new net N$88: R40.2, S10.1, S10.2
- new net N$89: R41.2, S11.1, S11.2
- new net N$90: R42.2, S12.1, S12.2
- new net N$91: R37.2, S7.1, S7.2
- new net N$92: C3.2, D2.A, Q1.C, SG1.1
- new net N$93: C9.1, Q1.B, R1.2, R2.2
- new net N$94: X1.ID_SC
- new net N$95: X1.ID_SD
- new net N$96: X1.CE1
- new net N$97: X1.CE0
- new net N$98: X1.MOSI
- new net N$99: X1.MISO
- new net PGC: R26.1, X1.GP4
- new net PGD: R25.1, X1.GP17
- new net UP: C20.1, R31.1, S8.3, S8.4, X1.GP25
- net AGND: now also C1.2, C10.2, C11.2, C12.2, C13.2, C14.2, C15.2, C16.2, C17.2, C18.2, C19.2, C2.2, C20.2, C21.2, C22.2, C23.2, C24.2, C25.2, C6.-, C7.2, C8.2, C9.2, JP11.1, Q1.E, Q5.E, Q6.E, Q7.E, R15.1, R16.1, R17.1, R18.1, R19.1, R2.1, R20.1, R21.1, R22.1, R23.1, R27.1, R28.1, R29.1, R37.1, R38.1, R39.1, R40.1, R41.1, R42.1, R43.1, X1.GND@14, X1.GND@20, X1.GND@25, X1.GND@30, X1.GND@34, X1.GND@39, X1.GND@6, X1.GND@9, Z1.A; no longer C31.-, JP78.2, JP79.1, JP80.1, JP80.2, JP81.1, JP81.2, JP82.1, JP82.2, LED1.C
- net VCC: now also C3.1, D2.C, L1.2, Q2.E, Q3.E, Q4.E, R10.2, R11.2, R9.2, SG1.2; no longer C31.+, JP78.1, JP79.2, R44.A, R49.2
Other:
- note added: "Alimentação"
- note added: "Botões"
- note added: "Buzzer"
- note added: "Conecotor GPIO"
- note added: "Conversor_PICProgrammer"
- note removed: "Conexão_Fonte"
