File: Conexão_Motor.sch (EAGLE design)
At the start: 74 parts

Commit message: Rev4 - Adição do circuito de Alta Latência - Previsão de conexão de módulos de expansão - Correção de falhas e previsão de melhorias com relação a estabilidade do sistema - Definição dos valores iniciais para cada componente - Previsão de circuito conversor de nivel para possivel feature implementável de atualização de firmware.
Parts:
- removed C1, C2: (no value), rcl:C-EUC0805K
- removed JP11: (no value), jumper:JP2E
- added C4, C5: 100nf/50V, rcl:C-EUC0805K
- added JP73: (no value), jumper:JP2E
- JP10, JP20, JP21: device jumper:JP2E -> jumper:JP1E
- JP2, JP3, JP4: device jumper:JP1E -> jumper:JP2E
- JP38, JP39, JP56, JP57: device jumper:JP2E -> jumper:JP8Q
- JP5, JP6, JP7, JP8: device jumper:JP8Q -> jumper:JP2E
Connections:
- net AGND: now also C4.2, C5.2, JP12.1, JP13.1, JP14.1, JP15.1, JP16.1, JP17.1, JP18.1, JP19.1, JP2.1, JP20.1, JP20.2, JP21.1, JP21.2, JP22.1, JP23.1, JP24.1, JP25.1, JP26.1, JP27.1, JP28.1, JP29.1, JP30.1, JP31.1, JP32.1, JP33.1, JP34.1, JP35.1, JP36.1, JP37.1, JP40.1, JP41.1, JP42.1, JP43.1, JP44.1, JP45.1, JP46.1, JP47.1, JP48.1, JP49.1, JP5.1, JP50.1, JP51.1, JP52.1, JP53.1, JP54.1, JP55.1, JP58.1, JP59.1, JP6.1, JP60.1, JP61.1, JP62.1, JP63.1, JP64.1, JP65.1, JP66.1, JP67.1, JP68.1, JP69.1, JP7.1, JP70.1, JP71.1, JP72.1, JP73.1, JP8.1; no longer C1.2, C2.2, JP3.2, JP4.2
- net M00: now also JP38.2; no longer JP8.2
- net M01: now also JP38.4, JP8.3; no longer JP8.4
- net M02: now also JP38.6, JP7.3; no longer JP8.6
- net M03: now also JP38.8, JP6.3; no longer JP8.8
- net M04: now also JP38.10, JP5.3; no longer JP8.10
- net M05: now also JP38.12, JP4.3; no longer JP8.12
- net M06: now also JP3.3, JP38.14; no longer JP8.14
- net M07: now also JP2.3, JP38.16; no longer JP8.16
- net M08: now also JP19.3, JP38.15; no longer JP8.15
- net M09: now also JP18.3, JP38.13; no longer JP8.13
- net M10: now also JP17.3, JP38.11; no longer JP8.11
- net M11: now also JP16.3, JP38.9; no longer JP8.9
- net M12: now also JP15.3, JP38.7; no longer JP8.7
- net M13: now also JP14.3, JP38.5; no longer JP8.5
- net M14: now also JP13.3, JP38.3; no longer JP8.3
- net M15: now also JP12.3, JP38.1; no longer JP8.1
- net M16: now also JP29.3, JP56.2; no longer JP7.2
- net M17: now also JP28.3, JP56.4; no longer JP7.4
- net M18: now also JP27.3, JP56.6; no longer JP7.6
- net M19: now also JP26.3, JP56.8; no longer JP7.8
- net M20: now also JP25.3, JP56.10; no longer JP7.10
- net M21: now also JP24.3, JP56.12; no longer JP7.12
- net M22: now also JP23.3, JP56.14; no longer JP7.14
- net M23: now also JP22.3, JP56.16; no longer JP7.16
- net M24: now also JP37.3, JP56.15; no longer JP7.15
- net M25: now also JP36.3, JP56.13; no longer JP7.13
- net M26: now also JP35.3, JP56.11; no longer JP7.11
- net M27: now also JP34.3, JP56.9; no longer JP7.9
- net M28: now also JP33.3, JP56.7; no longer JP7.7
- net M29: now also JP32.3, JP56.5; no longer JP7.5
- net M30: now also JP31.3, JP56.3; no longer JP7.3
- net M31: now also JP30.3, JP56.1; no longer JP7.1
- net M32: now also JP39.2, JP47.3; no longer JP6.2
- net M33: now also JP39.4, JP46.3; no longer JP6.4
- net M34: now also JP39.6, JP45.3; no longer JP6.6
- net M35: now also JP39.8, JP44.3; no longer JP6.8
- net M36: now also JP39.10, JP43.3; no longer JP6.10
- net M37: now also JP39.12, JP42.3; no longer JP6.12
- net M38: now also JP39.14, JP41.3; no longer JP6.14
- net M39: now also JP39.16, JP40.3; no longer JP6.16
- net M40: now also JP39.15, JP55.3; no longer JP6.15
- net M41: now also JP39.13, JP54.3; no longer JP6.13
- net M42: now also JP39.11, JP53.3; no longer JP6.11
- net M43: now also JP39.9, JP52.3; no longer JP6.9
- net M44: now also JP39.7, JP51.3; no longer JP6.7
- net M45: now also JP39.5, JP50.3; no longer JP6.5
- net M46: now also JP39.3, JP49.3; no longer JP6.3
- net M47: now also JP39.1, JP48.3; no longer JP6.1
- net M48: now also JP57.2, JP65.3; no longer JP5.2
- net M49: now also JP57.4, JP64.3; no longer JP5.4
- net M50: now also JP57.6, JP63.3; no longer JP5.6
- net M51: now also JP57.8, JP62.3; no longer JP5.8
- net M52: now also JP57.10, JP61.3; no longer JP5.10
- net M53: now also JP57.12, JP60.3; no longer JP5.12
- net M54: now also JP57.14, JP59.3; no longer JP5.14
- net M55: now also JP57.16, JP58.3; no longer JP5.16
- net M56: now also JP57.15, JP73.3; no longer JP5.15
- net M57: now also JP57.13, JP72.3; no longer JP5.13
- net M58: now also JP57.11, JP71.3; no longer JP5.11
- net M59: now also JP57.9, JP70.3; no longer JP5.9
- net M60: now also JP57.7, JP69.3; no longer JP5.7
- net M61: now also JP57.5, JP68.3; no longer JP5.5
- net M62: now also JP57.3, JP67.3; no longer JP5.3
- net M63: now also JP57.1, JP66.3; no longer JP5.1
- net VCC: now also C4.1, C5.1, JP10.1, JP10.2, JP12.2, JP13.2, JP14.2, JP15.2, JP16.2, JP17.2, JP18.2, JP19.2, JP22.2, JP23.2, JP24.2, JP25.2, JP26.2, JP27.2, JP28.2, JP29.2, JP3.2, JP30.2, JP31.2, JP32.2, JP33.2, JP34.2, JP35.2, JP36.2, JP37.2, JP4.2, JP40.2, JP41.2, JP42.2, JP43.2, JP44.2, JP45.2, JP46.2, JP47.2, JP48.2, JP49.2, JP5.2, JP50.2, JP51.2, JP52.2, JP53.2, JP54.2, JP55.2, JP58.2, JP59.2, JP6.2, JP60.2, JP61.2, JP62.2, JP63.2, JP64.2, JP65.2, JP66.2, JP67.2, JP68.2, JP69.2, JP7.2, JP70.2, JP71.2, JP72.2, JP73.2, JP8.2; no longer C1.1, C2.1, JP2.1
Other:
- moved on the sheet: JP1, JP12, JP13, JP14, JP15, JP16, JP17, JP18, JP19, JP22, JP23, JP24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
