File: DIDV_Full.sch (EAGLE design)
At the start: 284 parts, among them IC1 PIC18F4550_TQFP

Commit message: -  Inclusão do circuito de buzzer; -  Correção e prevenção contra ruídos nas linhas comunicação;
Parts:
- removed D1: BAS40, diode:BAS40
- removed Q1: (no value), crystal:CRYSTALHC49UP
- added C33, C34, C35, C36, C37, C38, C39, C40, C41, C42, C43, C44, C46: (no value), rcl:C-EUC0603K
- added C45: (no value), rcl:C-USC0805K
- added C47: (no value), rcl:C-EUC0805K
- added D5: BAS40, diode:BAS40
- added D6: BAS21, diode:BAS40
- added LSP1: LSP10, solpad:LSP10
- added Q3: (no value), crystal:CRYSTALHC49U-V
- added Q4: BC817, transistor-npn:BC817-16LT1SMD
- added R107, R108, R109, R110, R111, R112, R113: (no value), rcl:R-EU_R0603
- added SG2: F/CM12P, buzzer:F/CM12P
- added SJ6: JUMPER-PAD-3-2OF3_NC_BY_PASTE, SparkFun-Passives:JUMPER-PAD-3-2OF3_NC_BY_PASTE
- C16: device rcl:C-EUC0603K -> rcl:C-EUC0805
- C2: device rcl:C-EUC0805 -> rcl:C-EUC0805K
- C31, C32: device rcl:C-EUC0805K -> rcl:C-EUC0603K
- C4: device rcl:CPOL-EU140CLH-1014 -> rcl:C-EUC0805
- C5: device rcl:C-EUC0603K -> rcl:CPOL-EU140CLH-1014
- C6: device rcl:C-EUC0805 -> rcl:C-EUC0603K
- D2: value (none) -> BAS40; device diode:DIODE-SMC -> diode:BAS40
- D3: value BAS70 -> (none); device diode:BAS70 -> diode:DIODE-SMC
- D4: value BAS40 -> BAS70; device diode:BAS40 -> diode:BAS70
- Q2: device crystal:CRYSTALHC49U-V -> crystal:CRYSTALHC49UP
Connections:
- removed net N$43: IC1.RA2/AN2/VREF-/CVREF
- removed net N$9: C6.1, C7.1, D4.C, L1.1
- removed net VCC1: R106.2
- new net BUZZER: IC1.RB3/AN9/CCP2/VPO, SJ6.1
- new net N$10: C34.2, IC4.SIN, R109.2
- new net N$12: C35.2, IC5.SIN, R110.2
- new net N$13: IC5.SOUT, R111.1
- new net N$17: LSP1.MP, SJ6.3
- new net N$2: C7.1, C8.1, D5.C, L1.1
- new net N$23: C45.2, D6.A, Q4.C, SG2.1
- new net N$24: R112.1, SJ6.2
- new net N$25: C46.1, Q4.B, R112.2, R113.2
- new net N$3: C32.2, IC2.SIN, R107.2
- new net N$7: C33.2, IC3.SIN, R108.2
- net AGND: now also C32.1, C33.1, C34.1, C35.1, C36.2, C37.2, C38.2, C39.2, C4.2, C40.2, C41.2, C42.2, C43.2, C44.1, C46.2, C47.2, C5.-, D4.A, Q4.E, R113.1; no longer C32.2, C4.-, C5.2, D3.A
- net B00: now also C19.1; no longer C18.1
- net B01: now also C20.1; no longer C19.1
- net B02: now also C21.1; no longer C20.1
- net B03: now also C22.1; no longer C21.1
- net B04: now also C23.1; no longer C22.1
- net B05: now also C30.1; no longer C29.1
- net BACKSPACE: now also C25.1; no longer C24.1
- net DOWN: now also C31.1; no longer C30.1
- net ENTER: now also C24.1; no longer C23.1
- net ESC: now also C26.1; no longer C25.1
- net ESPAÇO: now also C27.1; no longer C26.1
- net FIM: now also C28.1, IC1.RA2/AN2/VREF-/CVREF; no longer C27.1, IC1.RB3/AN9/CCP2/VPO
- net GSCLK: now also C36.1, C37.1, C38.1, C39.1
- net N$109: now also D3.A; no longer D2.A
- net N$111: now also C6.1, D2.C; no longer C5.1, D1.C
- net N$112: now also D2.A; no longer D1.A
- net N$113: now also C4.1, C5.+, D4.C; no longer C2.1, C4.+, D2.C
- net N$114: now also D5.A; no longer D4.A
- net OSC1: now also C17.1, Q3.1; no longer C16.1, Q1.1
- net OSC2: now also C18.1, Q3.2; no longer C17.1, Q1.2
- net SCLK: now also C40.1, C41.1, C42.1, C43.1
- net SIN: now also R107.1; no longer IC2.SIN
- net SO2: now also R108.1; no longer IC3.SIN
- net SO3: now also R109.1; no longer IC4.SIN
- net SO4: now also R110.1; no longer IC5.SIN
- net SOUT: now also C44.2, R111.2; no longer IC5.SOUT
- net UP: now also C29.1; no longer C28.1
- net VCC: now also C16.1, C2.1, C45.1, C47.1, D6.C, R106.2, SG2.2; no longer C10.1, C31.1, C32.1
- net VUSB: now also C10.1; no longer C8.1
Other:
- note added: "On Raspberry Pi B+"
- moved on the sheet: C10, C11, C12, C13, C14, C15, C16, C17, C18, C19, C20, C21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

Commit message: Rev4 - Adição do circuito de Alta Latência - Previsão de conexão de módulos de expansão - Correção de falhas e previsão de melhorias com relação a estabilidade do sistema - Definição dos valores iniciais para cada componente - Previsão de circuito conversor de nivel para possivel feature implementável de atualização de firmware.
Parts:
- removed D3: (no value), diode:DIODE-SMC
- removed D5: BAS40, diode:BAS40
- removed SG2: F/CM12P, buzzer:F/CM12P
- removed SJ6: JUMPER-PAD-3-2OF3_NC_BY_PASTE, SparkFun-Passives:JUMPER-PAD-3-2OF3_NC_BY_PASTE
- added C48, C49, C50, C51, C52, C53, C54, C55: 100nf/50V, rcl:C-EUC0805
- added C56: 10nf/50V, rcl:C-EUC0603K
- added D1: S1J, diode:DIODE-SMC
- added D7, D8: BAS21, diode:BAS40
- added JP84: (no value), jumper:JP1E
- added JP85: (no value), jumper:JP7Q
- added JP86: (no value), jumper:JP1Q
- added K1: 4052, relay:4052
- added L3: 330m, inductor-neosid:MS50
- added LSP2, LSP3: LSP10, solpad:LSP10
- added Q1, Q10, Q5, Q6, Q7: BC817, transistor-npn:BC817-16LT1SMD
- added R114, R115, R116, R117, R118, R119, R120, R122, R124: (no value), rcl:R-US_R0805
- added R121, R123: 649, rcl:R-US_R0805
- added R125: 22, rcl:R-EU_R0603
- added R126: 10k, rcl:R-EU_R0603
- added R127, R128: 100, rcl:R-EU_R0603
- added R129: 100k, rcl:R-US_R0805
- added R130: 0r, rcl:R-EU_R0603
- added R131: 150k, rcl:R-EU_R0603
- added R132: 100k, rcl:R-EU_R0603
- added SG1: F/CM12P, buzzer:F/CM12P
- added X1: RASPBERRYPI-B+-GPIO, SparkFun-Boards:RASPBERRYPI-B+-GPIO
- added XT1: 20Mhz, crystal:CRYSTALHC49UP
- added XT2: (no value), crystal:CRYSTALHC49U-V
- added Z1, Z2: 5v1, diode:BAS70
- C1: value (none) -> 100nf/50V; device rcl:CPOL-EUE3.5-10 -> rcl:C-EUC0603K
- C10, C11, C12, C13, C14, C15: value (none) -> 1nf/50V; device rcl:C-EUC0805 -> rcl:C-EUC0603K
- C16, C3, C9: value (none) -> 10nf/50V; device rcl:C-EUC0805 -> rcl:C-EUC0603K
- C17, C18: value (none) -> 10nf/50V
- C19, C20, C21, C22, C23, C24, C25: value (none) -> 1nf/50V
- C2: value (none) -> 100nf/50V; device rcl:C-EUC0805K -> rcl:C-EUC0603K
- C26, C6: value (none) -> 470uf/35V; device rcl:C-EUC0603K -> rcl:CPOL-EU140CLH-1014
- C27, C28, C32, C33: value (none) -> 100nf/50V; device rcl:C-EUC0603K -> rcl:C-EUC0805
- C29, C30, C36, C37, C38, C39, C40, C41, C42, C43, C44, C46, C7, C8: value (none) -> 100nf/50V
- C31: value (none) -> 2200uf/35V; device rcl:C-EUC0603K -> rcl:CPOL-EUE3.5-10
- C34, C35: value (none) -> 22pf/50V
- C4: value (none) -> 100nf/50V; device rcl:C-EUC0805 -> rcl:C-EUC0805K
- C45: value (none) -> 100nf/50V; device rcl:C-USC0805K -> rcl:C-EUC0603K
- C47: value (none) -> 10nf/50V; device rcl:C-EUC0805K -> rcl:C-EUC0603K
- C5: value (none) -> 100nf/50V; device rcl:CPOL-EU140CLH-1014 -> rcl:C-EUC0805K
- D2: value BAS40 -> BAS21
- D4: value BAS70 -> S3J; device diode:BAS70 -> diode:DIODE-SMC
- F1: value (none) -> 5A/250V
- IC1: value PIC18F4550_TQFP -> (none); device microchip:PIC18F4550_TQFP -> TLC5940:IC-PACKAGE_DIL28-3
- IC5: value (none) -> PIC18F4550; device TLC5940:IC-PACKAGE_DIL28-3 -> microchip:PIC18F4550_TQFP
- JP11, JP75: device jumper:JP2E -> jumper:JP1Q
- JP12, JP13, JP14, JP15, JP2, JP3, JP4, JP5, JP6, JP7, JP8: device jumper:JP1E -> jumper:JP2E
- JP16, JP17, JP18, JP19: device jumper:JP8Q -> jumper:JP2E
- JP20, JP21, JP74, JP76, JP77, JP78, JP79, JP80, JP81, JP82: device jumper:JP2E -> jumper:JP1E
- JP38, JP39, JP56, JP57: device jumper:JP2E -> jumper:JP8Q
- JP9: device jumper:JP1Q -> jumper:JP2E
- L1, L2: value (none) -> 330m
- Q2: value (none) -> BC807; device crystal:CRYSTALHC49UP -> transistor-pnp:BC807-40SMD
- Q3: value (none) -> BC807; device crystal:CRYSTALHC49U-V -> transistor-pnp:BC807-40SMD
- Q4: value BC817 -> BC807; device transistor-npn:BC817-16LT1SMD -> transistor-pnp:BC807-40SMD
- R1: value (none) -> 150k; device rcl:R-US_0613/5V -> rcl:R-EU_R0603
- R10, R11, R12, R13, R14, R27, R28, R29, R9: value (none) -> 100k; device rcl:R-US_R0805 -> rcl:R-EU_R0603
- R100, R102, R103, R104, R105, R106, R107, R108, R109, R110, R111, R112, R113, R79, R80, R81, R83, R85, R87, R88, R89, R90, R91, R92, R93, R94, R95, R96, R97, R98: device rcl:R-EU_R0603 -> rcl:R-US_R0805
- R101, R99: value (none) -> 22
- R15, R16, R17, R18, R19, R20, R37, R38, R39, R40, R41, R42, R43: value (none) -> 100; device rcl:R-US_R0805 -> rcl:R-EU_R0603
- R2: value (none) -> 100k; device resistor-shunt:PMA-B -> rcl:R-EU_R0603
- R21, R22, R23, R30, R31, R32, R33, R34, R35, R36, R7, R8: value (none) -> 10k; device rcl:R-US_R0805 -> rcl:R-EU_R0603
- R24, R25, R26: value (none) -> 150k; device rcl:R-US_R0805 -> rcl:R-EU_R0603
- R3, R4, R5, R6: value (none) -> 10k
- R44: value (none) -> 4 m; device rcl:R-US_R0805 -> resistor-shunt:PMA-B
- R49: value (none) -> 470; device rcl:R-US_R0805 -> rcl:R-US_0613/5V
- R58, R60, R70, R77: value (none) -> 22; device rcl:R-US_R0805 -> rcl:R-EU_R0603
- R82, R84: value (none) -> 649; device rcl:R-EU_R0603 -> rcl:R-US_R0805
- R86: value (none) -> 1M
- SJ1: value JUMPER-PAD-2-NOYES_SILK -> JUMPER-PAD-3-2OF3_NC_BY_PASTE; device SparkFun-Passives:JUMPER-PAD-2-NOYES_SILK -> SparkFun-Passives:JUMPER-PAD-3-2OF3_NC_BY_PASTE
- SJ3: value JUMPER-PAD-3-2OF3_NC_BY_PASTE -> JUMPER-PAD-2-NOYES_SILK; device SparkFun-Passives:JUMPER-PAD-3-2OF3_NC_BY_PASTE -> SparkFun-Passives:JUMPER-PAD-2-NOYES_SILK
Connections:
- removed net B00: C19.1, IC1.RD0/SPP0, R91.1, S9.3, S9.4
- removed net N$1: R85.2, S3.1, S3.2
- removed net N$10: C34.2, IC4.SIN, R109.2
- removed net N$109: D3.A, JP9.2
- removed net N$110: R3.2, S13.1, S13.2
- removed net N$111: C6.1, D2.C, R89.2, S13.3, S13.4
- removed net N$112: D2.A, R4.1
- removed net N$113: C3.1, C4.1, C5.+, D3.C, D4.C, L2.1
- removed net N$114: D5.A, U1.VBUS
- removed net N$115: R6.2, U1.D+
- removed net N$116: R5.2, U1.D-
- removed net N$118: IC4.IREF, R57.2, R77.2
- removed net N$12: C35.2, IC5.SIN, R110.2
- removed net N$13: IC5.SOUT, R111.1
- removed net N$14: R79.2, S9.1, S9.2
- removed net N$144: IC2.IREF, R74.2, R75.2
- removed net N$17: LSP1.MP, SJ6.3
- removed net N$18: IC1.RE2/AN7/OESPP
- removed net N$19: IC1.RE1/AN6/CK2SPP
- removed net N$2: C7.1, C8.1, D5.C, L1.1
- removed net N$20: IC1.RE0/AN5/CK1SPP
- removed net N$21: IC1.RA5/AN4/!SS!/HLVDIN/C2OUT
- removed net N$22: IC1.RA4/T0CKI/CIOUT/RCV
- removed net N$23: C45.2, D6.A, Q4.C, SG2.1
- removed net N$24: R112.1, SJ6.2
- removed net N$25: C46.1, Q4.B, R112.2, R113.2
- removed net N$29: R84.2, S7.1, S7.2
- removed net N$3: C32.2, IC2.SIN, R107.2
- removed net N$30: R83.2, S8.1, S8.2
- removed net N$31: R82.2, S12.1, S12.2
- removed net N$36: IC1.RB4/AN11/KBI0/CSSPP
- removed net N$37: IC1.RB5/KBI1/PGM
- removed net N$38: R81.2, S11.1, S11.2
- removed net N$39: R80.2, S10.1, S10.2
- removed net N$4: LED1.A, R1.1
- removed net N$44: IC1.RA3/AN3/VREF+
- removed net N$5: F1.2, R2.B
- removed net N$6: F1.1, JP1.1, JP1.2, JP5.1, JP5.2, JP7.1, JP7.2
- removed net N$64: IC3.IREF, R23.2, R76.2
- removed net N$68: R98.2, S1.1, S1.2
- removed net N$69: R97.2, S2.1, S2.2
- removed net N$7: C33.2, IC3.SIN, R108.2
- removed net N$70: R88.2, S6.1, S6.2
- removed net N$71: R87.2, S5.1, S5.2
- removed net N$72: R86.2, S4.1, S4.2
- removed net N$8: R105.2, S14.1, S14.2
- removed net N$85: IC5.IREF, R40.2, R78.2
- new net +3V3: C1.1, C2.1, R3.2, R30.2, R31.2, R32.2, R33.2, R34.2, R35.2, R36.2, R4.2, R5.2, R6.2, R7.2, R8.2, X1.3.3V@1, X1.3.3V@17
- new net B06: C10.1, R3.1, S1.3, S1.4, X1.GP19
- new net EXP: IC5.RD4/SPP4, R131.2
- new net EXPA: JP85.4, K12.S
- new net EXPB: JP85.3, K13.P
- new net N$100: X1.SCLK
- new net N$101: X1.RXI
- new net N$102: X1.TXO
- new net N$103: X1.SCL
- new net N$104: X1.SDA
- new net N$105: Q7.C, R14.1
- new net N$106: C18.1, Q7.B, R26.2, R29.2
- new net N$107: Q4.B, R11.1, R14.2
- new net N$108: LSP3.MP, Q4.C, R23.2
- new net N$117: Q6.C, R13.1
- new net N$119: C17.1, Q6.B, R25.2, R28.2
- new net N$120: Q3.B, R10.1, R13.2
- new net N$121: LSP2.MP, Q3.C, R22.2
- new net N$122: Q5.C, R12.1
- new net N$123: C16.1, Q5.B, R24.2, R27.2
- new net N$124: Q2.B, R12.2, R9.1
- new net N$125: LSP1.MP, Q2.C, R21.2
- new net N$126: IC5.RE2/AN7/OESPP
- new net N$127: IC5.RE1/AN6/CK2SPP
- new net N$128: IC5.RE0/AN5/CK1SPP
- new net N$129: IC5.RA5/AN4/!SS!/HLVDIN/C2OUT
- new net N$130: IC5.RA4/T0CKI/CIOUT/RCV
- new net N$131: IC5.RB4/AN11/KBI0/CSSPP
- new net N$132: IC5.RB5/KBI1/PGM
- new net N$133: IC5.RA3/AN3/VREF+
- new net N$134: R127.2, S14.1, S14.2
- new net N$135: C47.1, D7.C, R128.2, S14.3, S14.4
- new net N$136: D7.A, R126.1
- new net N$137: D4.A, JP75.2
- new net N$138: C26.+, C27.1, C28.1, D4.C, L2.1, Z2.C
- new net N$139: R70.2, U1.D+
- new net N$140: R77.2, U1.D-
- new net N$141: D6.A, U1.VBUS
- new net N$142: IC1.IREF, R82.2, R83.2
- new net N$143: IC3.IREF, R121.2, R122.2
- new net N$145: IC4.IREF, R123.2, R124.2
- new net N$146: IC2.IREF, R84.2, R85.2
- new net N$147: C32.1, C33.1, D6.C, L3.1
- new net N$148: C30.2, IC2.SIN, R60.2
- new net N$149: C29.2, IC1.SIN, R58.2
- new net N$150: C37.2, IC4.SIN, R101.2
- new net N$151: C36.2, IC3.SIN, R99.2
- new net N$152: IC3.SOUT, R125.1
- new net N$153: IC5.RC1/T1OSI/ICCP2/!UOE
- new net N$154: IC5.RD0/SPP0
- new net N$155: IC5.RD1/SPP1
- new net N$156: IC5.RD2/SPP2
- new net N$157: IC5.RD3/SPP3
- new net N$158: IC5.RC6/TX/CK
- new net N$159: IC5.RC0/TIOSO/T13CKI
- new net N$160: IC5.RA2/AN2/VREF-/CVREF
- new net N$161: IC5.!MCLR!/VPP/RE3
- new net N$162: IC5.RB2/AN8/INT2/VMO
- new net N$163: IC5.RB3/AN9/CCP2/VPO
- new net N$164: IC5.RD7/SPP7/P1D
- new net N$165: IC5.RD6/SPP6/P1C
- new net N$166: Q10.C, R130.1
- new net N$167: C56.1, Q10.B, R131.1, R132.2
- new net N$168: D8.A, K11.2, R130.2
- new net N$169: K13.O
- new net N$170: LED1.A, R49.1
- new net N$171: F1.2, R44.B
- new net N$172: F1.1, JP74.1, JP74.2, JP76.1, JP76.2, JP77.1, JP77.2
- new net N$76: D1.A, JP11.2
- new net N$77: C6.+, C7.1, C8.1, D1.C, L1.1, Z1.C
- new net N$78: R20.2, S6.1, S6.2
- new net N$79: R15.2, S1.1, S1.2
- new net N$80: R16.2, S2.1, S2.2
- new net N$81: R17.2, S3.1, S3.2
- new net N$82: R18.2, S4.1, S4.2
- new net N$83: R19.2, S5.1, S5.2
- new net N$84: R43.2, S13.1, S13.2
- new net N$86: R38.2, S8.1, S8.2
- new net N$87: R39.2, S9.1, S9.2
- new net N$88: R40.2, S10.1, S10.2
- new net N$89: R41.2, S11.1, S11.2
- new net N$90: R42.2, S12.1, S12.2
- new net N$91: R37.2, S7.1, S7.2
- new net N$92: C3.2, D2.A, Q1.C, SG1.1
- new net N$93: C9.1, Q1.B, R1.2, R2.2
- new net N$94: X1.ID_SC
- new net N$95: X1.ID_SD
- new net N$96: X1.CE1
- new net N$97: X1.CE0
- new net N$98: X1.MOSI
- new net N$99: X1.MISO
- new net RA: IC5.RD5/SPP5/P1B, JP85.2, JP86.2, R129.1
- new net RB: JP85.1, JP86.1
- new net SOUT_: IC5.RB0/AN12/INT0/LFT0/SDI/SDA, K12.O, K13.S
- net AGND: now also C1.2, C26.-, C29.1, C30.1, C31.-, C32.2, C33.2, C34.2, C35.2, C36.1, C37.1, C38.1, C44.2, C45.2, C48.2, C49.2, C5.2, C50.2, C51.2, C52.2, C53.2, C54.2, C55.2, C56.2, C6.-, IC1.GND, IC5.VSS, IC5.VSS@1, JP12.1, JP13.1, JP16.1, JP17.1, JP18.1, JP19.1, JP20.2, JP21.1, JP21.2, JP22.1, JP23.1, JP24.1, JP25.1, JP26.1, JP27.1, JP28.1, JP29.1, JP3.1, JP30.1, JP31.1, JP32.1, JP33.1, JP34.1, JP35.1, JP36.1, JP37.1, JP40.1, JP41.1, JP42.1, JP43.1, JP44.1, JP45.1, JP46.1, JP47.1, JP48.1, JP49.1, JP5.1, JP50.1, JP51.1, JP52.1, JP53.1, JP54.1, JP55.1, JP58.1, JP59.1, JP60.1, JP61.1, JP62.1, JP63.1, JP64.1, JP65.1, JP66.1, JP67.1, JP68.1, JP69.1, JP7.1, JP70.1, JP71.1, JP72.1, JP73.1, JP75.1, JP78.2, JP79.1, JP80.1, JP80.2, JP81.1, JP81.2, JP82.1, JP82.2, JP83.1, JP85.11, JP85.13, Q1.E, Q10.E, Q5.E, Q6.E, Q7.E, R121.1, R122.1, R123.1, R124.1, R127.1, R132.1, R15.1, R16.1, R17.1, R18.1, R19.1, R2.1, R20.1, R21.1, R22.1, R27.1, R28.1, R29.1, R37.1, R38.1, R39.1, R41.1, R42.1, R43.1, X1.GND@14, X1.GND@20, X1.GND@25, X1.GND@30, X1.GND@34, X1.GND@39, X1.GND@6, X1.GND@9, Z1.A, Z2.A; no longer C1.-, C26.2, C29.2, C3.2, C30.2, C31.2, C32.1, C33.1, C34.1, C35.1, C36.2, C37.2, C38.2, C44.1, C5.-, C6.2, D4.A, IC1.VSS, IC1.VSS@1, IC5.GND, JP14.2, JP15.2, JP2.2, JP3.2, JP6.2, JP8.2, Q4.E, R105.1, R113.1, R3.1, R57.1, R74.1, R75.1, R76.1, R77.1, R78.1, R79.1, R80.1, R81.1, R86.1, R87.1, R88.1, R97.1, R98.1
- net B01: now also C15.1, R8.1, S6.3, S6.4, X1.GP5; no longer C20.1, IC1.RD1/SPP1, R92.1, S10.3, S10.4
- net B02: now also C14.1, R7.1, S5.3, S5.4, X1.GP6; no longer C21.1, IC1.RD2/SPP2, R93.1, S11.3, S11.4
- net B03: now also C13.1, R6.1, S4.3, S4.4, X1.GP12; no longer C22.1, IC1.RD3/SPP3, R94.1, S12.3, S12.4
- net B04: now also C12.1, R5.1, S3.3, S3.4, X1.GP13; no longer C23.1, IC1.RD4/SPP4, R95.1, S8.3, S8.4
- net B05: now also C11.1, R4.1, S2.3, S2.4, X1.GP16; no longer C30.1, IC1.RD5/SPP5/P1B, R96.1, S7.3, S7.4
- net BACKSPACE: now also C24.1, R35.1, S12.3, S12.4, X1.GP27; no longer C25.1, IC1.RC1/T1OSI/ICCP2/!UOE, R100.1, S4.3, S4.4
- net BLANK: now also IC1.BLANK, IC5.RA1/AN1, JP85.7, TP21.1, TP22.1, TP7.1, TP8.1; no longer IC1.RA1/AN1, IC5.BLANK, TP11.1, TP18.1, TP25.1, TP4.1
- net BUZZER: now also R1.1, X1.GP22; no longer IC1.RB3/AN9/CCP2/VPO, SJ6.1
- net D+: now also R70.1, SJ2.3; no longer R6.1, SJ4.3
- net D+_: now also IC5.RC5/D+/VP, SJ2.2; no longer IC1.RC5/D+/VP, SJ4.2
- net D-: now also R77.1, SJ1.3; no longer R5.1, SJ5.3
- net D-_: now also IC5.RC4/D-/VM, SJ1.2; no longer IC1.RC4/D-/VM, SJ5.2
- net DOWN: now also C19.1, R30.1, S7.3, S7.4, X1.GP24; no longer C31.1, IC1.RD7/SPP7/P1D, R106.1, S14.3, S14.4
- net ENTER: now also C25.1, R36.1, S13.3, S13.4, X1.GP26; no longer C24.1, IC1.RC0/TIOSO/T13CKI, R99.1, S3.3, S3.4
- net ESC: now also C23.1, R34.1, S11.3, S11.4, X1.GP20; no longer C26.1, IC1.RB2/AN8/INT2/VMO, R101.1, S5.3, S5.4
- net ESPAÇO: now also C22.1, R33.1, S10.3, S10.4, X1.GP21; no longer C27.1, IC1.RC6/TX/CK, R102.1, S6.3, S6.4
- net FIM: now also C21.1, R32.1, S9.3, S9.4, X1.GP23; no longer C28.1, IC1.RA2/AN2/VREF-/CVREF, R103.1, S2.3, S2.4
- net GSCLK: now also C43.1, C44.1, C45.1, C46.1, IC1.GSCLK, IC5.RC2/CCP1/P1A, JP85.5, TP11.1, TP12.1, TP25.1, TP26.1; no longer C36.1, C37.1, C38.1, C39.1, IC1.RC2/CCP1/P1A, IC5.GSCLK, TP13.1, TP20.1, TP27.1, TP6.1
- net M00: now also JP38.2, JP9.3, R46.1; no longer JP19.2, JP20.3, R58.1
- net M01: now also JP38.4, JP8.3, R48.1; no longer JP19.4, R59.1
- net M02: now also JP38.6, JP7.3, R51.1; no longer JP19.6, R60.1
- net M03: now also JP38.8, JP6.3, R53.1; no longer JP19.8, R61.1
- net M04: now also JP38.10, JP5.3, R55.1; no longer JP19.10, R62.1
- net M05: now also JP38.12, JP4.3, R57.1; no longer JP19.12, R63.1
- net M06: now also JP3.3, JP38.14, R61.1; no longer JP19.14, R64.1
- net M07: now also JP2.3, JP38.16, R63.1; no longer JP19.16, R65.1
- net M08: now also JP19.3, JP38.15, R65.1; no longer JP19.15, R66.1
- net M09: now also JP18.3, JP38.13; no longer JP19.13
- net M10: now also JP17.3, JP38.11, R69.1; no longer JP19.11, R68.1
- net M11: now also JP16.3, JP38.9, R72.1; no longer JP19.9, R69.1
- net M12: now also JP15.3, JP38.7, R74.1; no longer JP19.7, R70.1
- net M13: now also JP14.3, JP38.5, R76.1; no longer JP19.5, R71.1
- net M14: now also JP13.3, JP38.3, R79.1; no longer JP19.3, R72.1
- net M15: now also JP12.3, JP38.1, R81.1; no longer JP19.1, R73.1
- net M16: now also IC1.OUT0, JP29.3, JP56.2, R45.1; no longer IC3.OUT0, JP18.2, R7.1
- net M17: now also IC1.OUT1, JP28.3, JP56.4, R47.1; no longer IC3.OUT1, JP18.4, R8.1
- net M18: now also IC1.OUT2, JP27.3, JP56.6, R50.1; no longer IC3.OUT2, JP18.6, R9.1
- net M19: now also IC1.OUT3, JP26.3, JP56.8, R52.1; no longer IC3.OUT3, JP18.8, R10.1
- net M20: now also IC1.OUT4, JP25.3, JP56.10, R54.1; no longer IC3.OUT4, JP18.10, R11.1
- net M21: now also IC1.OUT5, JP24.3, JP56.12, R56.1; no longer IC3.OUT5, JP18.12, R12.1
- net M22: now also IC1.OUT6, JP23.3, JP56.14, R59.1; no longer IC3.OUT6, JP18.14, R13.1
- net M23: now also IC1.OUT7, JP22.3, JP56.16, R62.1; no longer IC3.OUT7, JP18.16, R14.1
- net M24: now also IC1.OUT8, JP37.3, JP56.15, R64.1; no longer IC3.OUT8, JP18.15, R15.1
- net M25: now also IC1.OUT9, JP36.3, JP56.13, R66.1; no longer IC3.OUT9, JP18.13, R16.1
- net M26: now also IC1.OUT10, JP35.3, JP56.11, R68.1; no longer IC3.OUT10, JP18.11, R17.1
- net M27: now also IC1.OUT11, JP34.3, JP56.9, R71.1; no longer IC3.OUT11, JP18.9, R18.1
- net M28: now also IC1.OUT12, JP33.3, JP56.7, R73.1; no longer IC3.OUT12, JP18.7, R19.1
- net M29: now also IC1.OUT13, JP32.3, JP56.5, R75.1; no longer IC3.OUT13, JP18.5, R20.1
- net M30: now also IC1.OUT14, JP31.3, JP56.3, R78.1; no longer IC3.OUT14, JP18.3, R21.1
- net M31: now also IC1.OUT15, JP30.3, JP56.1, R80.1; no longer IC3.OUT15, JP18.1, R22.1
- net M32: now also JP39.2, JP47.3, R88.1; no longer JP17.2, R41.1
- net M33: now also JP39.4, JP46.3, R90.1; no longer JP17.4, R42.1
- net M34: now also JP39.6, JP45.3, R92.1; no longer JP17.6, R43.1
- net M35: now also JP39.8, JP44.3, R94.1; no longer JP17.8, R44.1
- net M36: now also JP39.10, JP43.3, R96.1; no longer JP17.10, R45.1
- net M37: now also JP39.12, JP42.3, R98.1; no longer JP17.12, R46.1
- net M38: now also JP39.14, JP41.3, R102.1; no longer JP17.14, R47.1
- net M39: now also JP39.16, JP40.3, R104.1; no longer JP17.16, R48.1
- net M40: now also JP39.15, JP55.3, R106.1; no longer JP17.15, R49.1
- net M41: now also JP39.13, JP54.3, R108.1; no longer JP17.13, R50.1
- net M42: now also JP39.11, JP53.3, R110.1; no longer JP17.11, R51.1
- net M43: now also JP39.9, JP52.3, R112.1; no longer JP17.9, R52.1
- net M44: now also JP39.7, JP51.3, R114.1; no longer JP17.7, R53.1
- net M45: now also JP39.5, JP50.3, R116.1; no longer JP17.5, R54.1
- net M46: now also JP39.3, JP49.3, R118.1; no longer JP17.3, R55.1
- net M47: now also JP39.1, JP48.3, R120.1; no longer JP17.1, R56.1
- net M48: now also IC3.OUT0, JP57.2, JP65.3, R87.1; no longer IC5.OUT0, JP16.2, R24.1
- net M49: now also IC3.OUT1, JP57.4, JP64.3, R89.1; no longer IC5.OUT1, JP16.4, R25.1
- net M50: now also IC3.OUT2, JP57.6, JP63.3, R91.1; no longer IC5.OUT2, JP16.6, R26.1
- net M51: now also IC3.OUT3, JP57.8, JP62.3, R93.1; no longer IC5.OUT3, JP16.8, R27.1
- net M52: now also IC3.OUT4, JP57.10, JP61.3, R95.1; no longer IC5.OUT4, JP16.10, R28.1
- net M53: now also IC3.OUT5, JP57.12, JP60.3, R97.1; no longer IC5.OUT5, JP16.12, R29.1
- net M54: now also IC3.OUT6, JP57.14, JP59.3, R100.1; no longer IC5.OUT6, JP16.14, R30.1
- net M55: now also IC3.OUT7, JP57.16, JP58.3, R103.1; no longer IC5.OUT7, JP16.16, R31.1
- net M56: now also IC3.OUT8, JP57.15, JP73.3, R105.1; no longer IC5.OUT8, JP16.15, R32.1
- net M57: now also IC3.OUT9, JP57.13, JP72.3, R107.1; no longer IC5.OUT9, JP16.13, R33.1
- net M58: now also IC3.OUT10, JP57.11, JP71.3, R109.1; no longer IC5.OUT10, JP16.11, R34.1
- net M59: now also IC3.OUT11, JP57.9, JP70.3, R111.1; no longer IC5.OUT11, JP16.9, R35.1
- net M60: now also IC3.OUT12, JP57.7, JP69.3, R113.1; no longer IC5.OUT12, JP16.7, R36.1
- net M61: now also IC3.OUT13, JP57.5, JP68.3, R115.1; no longer IC5.OUT13, JP16.5, R37.1
- net M62: now also IC3.OUT14, JP57.3, JP67.3, R117.1; no longer IC5.OUT14, JP16.3, R38.1
- net M63: now also IC3.OUT15, JP57.1, JP66.3, R119.1; no longer IC5.OUT15, JP16.1, R39.1
- net MCLR: now also JP84.1, R24.1, SJ3.1, X1.GP18#; no longer JP10.1, SJ1.1
- net NC: now also IC1.XERR; no longer IC5.XERR
- net OSC1: now also C34.1, IC5.OSC1/CLKI, R86.2, XT1.1, XT2.1; no longer C17.1, IC1.OSC1/CLKI, Q2.1, Q3.1, R90.2
- net OSC2: now also C35.1, IC5.RA6/OSC2/CLKO, R86.1, XT1.2, XT2.2; no longer C18.1, IC1.RA6/OSC2/CLKO, Q2.2, Q3.2, R90.1
- net PGC: now also IC5.RB6/KBI2/PGC, R26.1, SJ4.2, X1.GP4; no longer IC1.RB6/KBI2/PGC, SJ2.2
- net PGC_OUT: now also JP83.3, SJ4.3; no longer JP11.3, SJ2.3
- net PGD: now also IC5.RB7/BKI3/PGD, R25.1, SJ5.2, X1.GP17; no longer IC1.RB7/BKI3/PGD, SJ3.2
- net PGD_OUT: now also JP83.2, SJ5.3; no longer JP11.2, SJ3.3
- net RB6: now also SJ4.1; no longer SJ2.1
- net RB7: now also SJ5.1; no longer SJ3.1
- net RC4: now also SJ1.1; no longer SJ5.1
- net RC5: now also SJ2.1; no longer SJ4.1
- net RESET: now also R128.1, SJ3.2; no longer IC1.!MCLR!/VPP/RE3, R89.1, SJ1.2
- net SCLK: now also C39.1, IC1.SCLK, IC5.RB1/AN10/INT1/SCK/SCL, JP85.6, TP17.1, TP18.1, TP3.1, TP4.1; no longer C43.1, IC1.RB1/AN10/INT1/SCK/SCL, IC5.SCLK, TP16.1, TP2.1, TP23.1, TP9.1
- net SHUNT_1: now also R44.SB; no longer R2.SB
- net SHUNT_2: now also R44.SA; no longer R2.SA
- net SIN: now also IC5.RC7/RX/DT/SDO, R60.1, TP2.1; no longer IC1.RC7/RX/DT/SDO, R107.1, TP1.1
- net SO2: now also R58.1, TP1.1, TP14.1; no longer R108.1, TP7.1, TP8.1
- net SO3: now also IC1.SOUT, R101.1, TP13.1, TP16.1; no longer IC3.SOUT, R109.1, TP14.1, TP15.1
- net SO4: now also R99.1, TP15.1, TP27.1; no longer R110.1, TP21.1, TP22.1
- net SOUT: now also C38.2, K12.P, R125.2; no longer C44.2, IC1.RB0/AN12/INT0/LFT0/SDI/SDA, R111.2
- net UP: now also C20.1, R31.1, S8.3, S8.4, X1.GP25; no longer C29.1, IC1.RD6/SPP6/P1C, R104.1, S1.3, S1.4
- net VCC: now also C3.1, C31.+, C4.1, C48.1, C49.1, C5.1, C50.1, C51.1, C52.1, C53.1, D2.C, D8.C, IC1.DCPRG, IC1.VCC, IC1.VPRG, IC5.VDD, IC5.VDD@1, JP1.1, JP1.2, JP10.1, JP14.2, JP15.2, JP16.2, JP17.2, JP18.2, JP19.2, JP2.2, JP22.2, JP23.2, JP24.2, JP25.2, JP26.2, JP27.2, JP28.2, JP29.2, JP3.2, JP30.2, JP31.2, JP32.2, JP33.2, JP34.2, JP35.2, JP36.2, JP37.2, JP40.2, JP41.2, JP42.2, JP43.2, JP44.2, JP45.2, JP46.2, JP47.2, JP48.2, JP49.2, JP5.2, JP50.2, JP51.2, JP52.2, JP53.2, JP54.2, JP55.2, JP58.2, JP59.2, JP6.2, JP60.2, JP61.2, JP62.2, JP63.2, JP64.2, JP65.2, JP66.2, JP67.2, JP68.2, JP69.2, JP7.2, JP70.2, JP71.2, JP72.2, JP73.2, JP78.1, JP79.2, JP8.2, JP84.2, JP85.12, JP85.14, JP9.2, K11.1, L3.2, Q2.E, Q3.E, Q4.E, R105.2, R107.2, R108.2, R109.2, R110.2, R111.2, R112.2, R113.2, R114.2, R115.2, R116.2, R117.2, R118.2, R119.2, R120.2, R126.2, R129.2, R44.A, R57.2, R74.2, R75.2, R76.2, R78.2, R79.2, R80.2, R81.2, R87.2, R88.2, R89.2, R90.2, R97.2, R98.2, SG1.2, TP10.1, TP23.1, TP24.1, TP9.1; no longer C1.+, C11.1, C12.1, C13.1, C14.1, C15.1, C16.1, C2.1, C45.1, C47.1, D6.C, IC1.VDD, IC1.VDD@1, IC5.DCPRG, IC5.VCC, IC5.VPRG, JP12.1, JP13.1, JP20.2, JP3.1, R1.2, R101.2, R12.2, R13.2, R14.2, R15.2, R16.2, R17.2, R18.2, R19.2, R2.A, R20.2, R21.2, R22.2, R24.2, R25.2, R26.2, R27.2, R28.2, R29.2, R30.2, R31.2, R32.2, R33.2, R34.2, R35.2, R36.2, R37.2, R38.2, R39.2, R4.2, R41.2, R42.2, R43.2, R44.2, R58.2, R60.2, R7.2, R70.2, R8.2, R99.2, SG2.2, TP12.1, TP19.1, TP26.1, TP5.1
- net VUSB: now also C54.1, C55.1, IC5.VUSB; no longer C10.1, C9.1, IC1.VUSB
- net XLAT: now also IC1.XLAT, IC5.RA0/AN0, JP85.8, TP19.1, TP20.1, TP5.1, TP6.1; no longer IC1.RA0/AN0, IC5.XLAT, TP10.1, TP17.1, TP24.1, TP3.1
Other:
- note added: "16x10k"
- note added: "Buzzer"
- note added: "Conecotor GPIO"
- note added: "Conversor_PICProgrammer"
- note added: "Seletor_de_Expansão"
- note removed: "On Raspberry Pi B+"

Commit message: Rev005
-  Inclusão de resistor série na linha do oscilador;
-  Nomenclatura correta dos componentes e nets;
-  Correção dos valores dos componentes.
Parts:
- added R133: 200, rcl:R-EU_R0603
Connections:
- net OSC2: now also R133.1, R133.2
