File: DIDV_-_Expansao_10.sch (EAGLE design)
At the start: 161 parts, among them U101 TLC5940QPWPREP, U201 TLC5940QPWPREP, U301 TLC5940QPWPREP, U401 TLC5940QPWPREP

Commit message: Revisão 7:
-  Alterações necessárias para adequação às necessidades dos exemplos de controle que temos.
-  Revisão da forma de filtragem de sinais digitais
-  Algumas nomenclaturas ainda estão erradas, deverão ser corrigidas com o andamento da implementação.
Parts:
- removed R122, R123, R125, R126, R225, R325, R426: (no value), rcl:R-US_R0805
- removed R124, R222, R223, R224, R322, R323, R324, R422, R423, R424, R425: 22, rcl:R-US_R0603
- removed R221, R321: 649, rcl:R-US_R0805
- removed TP101, TP102, TP103, TP104, TP105, TP17, TP18, TP19, TP20: TEST-POINT3X4, SparkFun-Passives:TEST-POINT3X4
- added C106, C206, C306, C407: 100pf/50V, rcl:C-EUC0603K
- added TP22, TP23, TP24, TP25, TP26, TP29, TP32, TP33, TP34, TP35, TP36, TP37, TP39: TEST-POINT3X4, SparkFun-Passives:TEST-POINT3X4
- R101: value 100k -> (none)
- R102, R104, R105, R106, R220, R320: value 22 -> (none); device rcl:R-US_R0603 -> rcl:R-US_R0805
- R103, R421: value 649 -> (none)
- R115, R419: value 10k -> 22
- R117: value 10k -> (none); device rcl:R-US_R0603 -> rcl:R-US_R0805
- R118: value (none) -> 649
- R119: value (none) -> 100k
- R120: value (none) -> 10k; device rcl:R-US_R0805 -> rcl:R-US_R0603
- R218, R318, R418: value 10k -> 649; device rcl:R-US_R0603 -> rcl:R-US_R0805
- R420: value 22 -> 10k
- renumbered TP106 to TP27, TP107 to TP28, TP21 to TP38
Connections:
- removed net BLANK: JP101.7, R106.1, R224.1, R324.1, R424.1, TP103.1, TP11.1, TP18.1, TP4.1
- removed net GSCLK: JP101.5, R105.1, R223.1, R323.1, R423.1, TP102.1, TP12.1, TP19.1, TP5.1
- removed net IR501: R421.2, R426.2, U401.IREF
- removed net N$13: C205.2, R215.2, U201.SIN
- removed net N$18: R219.2, U201.VPRG
- removed net N$22: C202.2, R222.2, U201.SCLK
- removed net N$24: R223.2, U201.GSCLK
- removed net N$30: R105.2, U101.GSCLK
- removed net N$35: C204.2, R224.2, U201.BLANK
- removed net N$36: C201.2, R220.2, U201.XLAT
- removed net N$41: R218.2, U201.DCPRG
- removed net N$42: C305.2, R315.2, U301.SIN
- removed net N$43: C105.2, R124.2, U101.SIN
- removed net N$45: TP14.1, U301.XERR
- removed net N$46: R319.2, U301.VPRG
- removed net N$47: R117.2, U101.VPRG
- removed net N$48: C104.2, R106.2, U101.BLANK
- removed net N$49: C101.2, R102.2, U101.XLAT
- removed net N$5 (its old number): C102.2, R104.2, U101.SCLK
- removed net N$50: C302.2, R322.2, U301.SCLK
- removed net N$51: R323.2, U301.GSCLK
- removed net N$52: C304.2, R324.2, U301.BLANK
- removed net N$53: C301.2, R320.2, U301.XLAT
- removed net N$54: R318.2, U301.DCPRG
- removed net N$55: C405.2, R415.2, U401.SIN
- removed net N$57: R419.2, U401.VPRG
- removed net N$58: C402.2, R422.2, U401.SCLK
- removed net N$59: R423.2, U401.GSCLK
- removed net N$60: C404.2, R424.2, U401.BLANK
- removed net N$61: C401.2, R420.2, U401.XLAT
- removed net N$62: R418.2, U401.DCPRG
- removed net N$63: R425.1, U401.SOUT
- removed net N$64: R115.2, U101.DCPRG
- removed net SCLK: C103.2, C203.2, C303.2, C403.2, JP101.6, R104.1, R222.1, R322.1, R422.1, TP101.1, TP16.1, TP2.1, TP9.1
- removed net XLAT: JP101.8, R102.1, R220.1, R320.1, R420.1, TP10.1, TP104.1, TP17.1, TP3.1
- new net BLANK_: C104.2, C204.2, C304.2, C404.2, JP101.7, TP12.1, TP25.1, TP35.1, TP4.1, U101.BLANK, U201.BLANK, U301.BLANK, U401.BLANK
- new net GSCLK_: C105.2, C205.2, C305.2, C405.2, JP101.5, TP13.1, TP26.1, TP36.1, TP5.1, U101.GSCLK, U201.GSCLK, U301.GSCLK, U401.GSCLK
- new net IR101: R118.2, R121.2, U101.IREF
- new net N$1: R120.2, U101.DCPRG
- new net N$11: R319.2, U301.DCPRG
- new net N$2: JP101.9
- new net N$3: C201.2, R215.2, U201.SIN
- new net N$39: C401.2, R415.2, U401.SIN
- new net N$4: C101.2, R115.2, U101.SIN
- new net N$6: R219.2, U201.DCPRG
- new net N$69: R420.2, U401.DCPRG
- new net N$71: R419.1, U401.SOUT
- new net N$8: C301.2, R315.2, U301.SIN
- new net N$9: TP15.1, U301.XERR
- new net SCLK_: C106.2, C206.2, C306.2, C407.2, JP101.6, TP10.1, TP2.1, TP23.1, TP33.1, U101.SCLK, U201.SCLK, U301.SCLK, U401.SCLK
- new net VPRG_: C102.2, C202.2, C302.2, C402.2, JP101.10, TP16.1, TP29.1, TP39.1, TP8.1, U101.VPRG, U201.VPRG, U301.VPRG, U401.VPRG
- new net XLAT_: C403.2, JP101.8, TP11.1, TP24.1, TP3.1, TP34.1, U101.XLAT, U201.XLAT, U301.XLAT, U401.XLAT
- net AGND: now also C106.1, C206.1, C306.1, C407.1, R118.1, R121.1, R218.1, R220.1, R318.1, R320.1, R418.1; no longer R103.1, R108.1, R221.1, R225.1, R321.1, R325.1, R426.1
- net EXPA: now also R115.1, TP22.1; no longer R124.1, TP105.1
- net EXPB: now also R419.2, TP37.1; no longer R425.2, TP20.1
- net F1: now also JP101.12; no longer JP101.10
- net F2: now also JP101.11; no longer JP101.9
- net IR201: now also R218.2, R220.2, U201.IREF; no longer R103.2, R108.2, U101.IREF
- net IR301: now also R318.2, R320.2, U301.IREF; no longer R221.2, R225.2, U201.IREF
- net IR401: now also R418.2, R421.2, U401.IREF; no longer R321.2, R325.2, U301.IREF
- net M00: now also R101.1; no longer R107.1
- net M01: now also R102.1; no longer R109.1
- net M02: now also R103.1; no longer R110.1
- net M03: now also R104.1; no longer R111.1
- net M04: now also R105.1; no longer R112.1
- net M05: now also R106.1; no longer R113.1
- net M06: now also R107.1; no longer R114.1
- net M07: now also R108.1; no longer R116.1
- net M08: now also R109.1; no longer R118.1
- net M09: now also R110.1; no longer R119.1
- net M10: now also R111.1; no longer R120.1
- net M11: now also R112.1; no longer R121.1
- net M12: now also R113.1; no longer R122.1
- net M13: now also R114.1; no longer R123.1
- net M14: now also R116.1; no longer R125.1
- net M15: now also R117.1; no longer R126.1
- net RA: now also R119.2; no longer R101.2
- net RB: now also R119.1; no longer R101.1
- net SOUT201: now also TP9.1; no longer TP8.1
- net SOUT301: now also TP14.1, TP32.1; no longer TP13.1, TP15.1
- net VCC: now also R101.2, R102.2, R103.2, R104.2, R105.2, R106.2, R108.2, R117.2, R120.1, R420.1; no longer R115.1, R117.1, R118.2, R119.2, R120.2, R121.2, R122.2, R123.2, R125.2, R126.2, R218.1, R318.1, R418.1, R419.1
Other:
- note added: "07"
- note added: "Iref - U101"
- note added: "Iref - U501"
- note removed: "06"
- note removed: "Iref - U100"
- moved on the sheet: JP101, R101, R102, R103, R104, R105, R106, R107, R108, R109, R110, R111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

Commit message: Revisão 8:
-  Add Circuito Buck
-  Alterações funcionais
-   Inserção dos primeiros boards
Other:
- note added: "08"
- note removed: "07"
Changed lines of the file:
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@@
 <text x="203.2" y="29.464" size="1.778" layer="150" font="vector">Dispositivo de Interface para</text>
 <text x="210.82" y="26.162" size="1.778" layer="150" font="vector">Deficientes Visuais</text>
-<text x="250.698" y="10.16" size="2.54" layer="150" font="vector">07</text>
+<text x="250.698" y="10.16" size="2.54" layer="150" font="vector">08</text>
 <text x="40.64" y="154.94" size="1.778" layer="97">16x10k</text>
 <text x="20.32" y="17.78" size="2.54" layer="150" font="vector">Iref - U101</text>
@@
 <text x="203.2" y="29.464" size="1.778" layer="150" font="vector">Dispositivo de Interface para</text>
 <text x="210.82" y="26.162" size="1.778" layer="150" font="vector">Deficientes Visuais</text>
-<text x="250.698" y="10.16" size="2.54" layer="150" font="vector">07</text>
+<text x="250.698" y="10.16" size="2.54" layer="150" font="vector">08</text>
 <text x="40.64" y="154.94" size="1.778" layer="97">16x10k</text>
 <text x="20.32" y="17.78" size="2.54" layer="150" font="vector">Iref - U101</text>
@@
 <text x="203.2" y="29.464" size="1.778" layer="150" font="vector">Dispositivo de Interface para</text>
 <text x="210.82" y="26.162" size="1.778" layer="150" font="vector">Deficientes Visuais</text>
-<text x="250.698" y="10.16" size="2.54" layer="150" font="vector">07</text>
+<text x="250.698" y="10.16" size="2.54" layer="150" font="vector">08</text>
 <text x="40.64" y="154.94" size="1.778" layer="97">16x10k</text>
 <text x="20.32" y="17.78" size="2.54" layer="150" font="vector">Iref - U101</text>
@@
 <text x="203.2" y="29.464" size="1.778" layer="150" font="vector">Dispositivo de Interface para</text>
 <text x="210.82" y="26.162" size="1.778" layer="150" font="vector">Deficientes Visuais</text>
-<text x="250.698" y="10.16" size="2.54" layer="150" font="vector">07</text>
+<text x="250.698" y="10.16" size="2.54" layer="150" font="vector">08</text>
 <text x="40.64" y="154.94" size="1.778" layer="97">16x10k</text>
 <text x="20.32" y="17.78" size="2.54" layer="150" font="vector">Iref - U501</text>

Commit message: Revisão 9
- Corrigidos algumas falhas de ligação
- Implementação com VPRG dos TLCs via Hardware
- Inserção do cálculo do Riref

Obs. Se somente a criação de boards, não será incrementado. No caso, se criado um board novo board vou subir para 9.1 e assim por diante.
Parts:
- removed C106, C206, C306, C407: 100pf/50V, rcl:C-EUC0603K
- removed TP16, TP29, TP39, TP8: TEST-POINT3X4, SparkFun-Passives:TEST-POINT3X4
- added R122, R221, R321, R422: (no value), rcl:R-US_R0805
- R101, R121, R201, R220, R301, R320, R401, R421: value (none) -> 10k; device rcl:R-US_R0805 -> rcl:R-US_R0603
- R115, R215, R315, R415: value 22 -> (none); device rcl:R-US_R0603 -> rcl:R-US_R0805
- R116, R216, R316, R416: value (none) -> 22; device rcl:R-US_R0805 -> rcl:R-US_R0603
- R118: value 649 -> 100k
- R119: value 100k -> (none)
- R120, R219, R319: value 10k -> RX; device rcl:R-US_R0603 -> rcl:R-US_R0805
- R218, R318, R418: value 649 -> (none)
- R419: value 22 -> RX; device rcl:R-US_R0603 -> rcl:R-US_R0805
- R420: value 10k -> 22
Connections:
- net AGND: now also R101.2, R120.1, R122.1, R201.2, R219.1, R221.1, R301.2, R319.1, R321.1, R401.2, R419.1, R422.1; no longer C106.1, C206.1, C306.1, C407.1, R118.1, R121.1, R218.1, R220.1, R318.1, R320.1, R418.1, R421.1
- net BLANK_: now also C103.2, C203.2, C303.2, C403.2; no longer C104.2, C204.2, C304.2, C404.2
- net EXPA: now also R116.1; no longer R115.1
- net EXPB: now also C405.2, R420.2; no longer C406.2, R419.2
- net GSCLK_: now also C104.2, C204.2, C304.2, C404.2; no longer C105.2, C205.2, C305.2, C405.2
- net IR101: now also R120.2, R122.2; no longer R118.2, R121.2
- net IR201: now also R219.2, R221.2; no longer R218.2, R220.2
- net IR301: now also R319.2, R321.2; no longer R318.2, R320.2
- net IR401: now also R419.2, R422.2; no longer R418.2, R421.2
- net M00: now also R102.1, R202.1, R302.1, R402.1; no longer R101.1, R201.1, R301.1, R401.1
- net M01: now also R103.1, R203.1, R303.1, R403.1; no longer R102.1, R202.1, R302.1, R402.1
- net M02: now also R104.1, R204.1, R304.1, R404.1; no longer R103.1, R203.1, R303.1, R403.1
- net M03: now also R105.1, R205.1, R305.1, R405.1; no longer R104.1, R204.1, R304.1, R404.1
- net M04: now also R106.1, R206.1, R306.1, R406.1; no longer R105.1, R205.1, R305.1, R405.1
- net M05: now also R107.1, R207.1, R307.1, R407.1; no longer R106.1, R206.1, R306.1, R406.1
- net M06: now also R108.1, R208.1, R308.1, R408.1; no longer R107.1, R207.1, R307.1, R407.1
- net M07: now also R109.1, R209.1, R309.1, R409.1; no longer R108.1, R208.1, R308.1, R408.1
- net M08: now also R110.1, R210.1, R310.1, R410.1; no longer R109.1, R209.1, R309.1, R409.1
- net M09: now also R111.1, R211.1, R311.1, R411.1; no longer R110.1, R210.1, R310.1, R410.1
- net M10: now also R112.1, R212.1, R312.1, R412.1; no longer R111.1, R211.1, R311.1, R411.1
- net M11: now also R113.1, R213.1, R313.1, R413.1; no longer R112.1, R212.1, R312.1, R412.1
- net M12: now also R114.1, R214.1, R314.1, R414.1; no longer R113.1, R213.1, R313.1, R413.1
- net M13: now also R115.1, R215.1, R315.1, R415.1; no longer R114.1, R214.1, R314.1, R414.1
- net M14: now also R117.1, R217.1, R317.1, R417.1; no longer R116.1, R216.1, R316.1, R416.1
- net M15: now also R119.1, R218.1, R318.1, R418.1; no longer R117.1, R217.1, R317.1, R417.1
- net N$1: now also R121.2; no longer R120.2
- net N$11: now also R320.2; no longer R319.2
- net N$3: now also R216.2; no longer R215.2
- net N$39: now also R416.2; no longer R415.2
- net N$4: now also R116.2; no longer R115.2
- net N$6: now also R220.2; no longer R219.2
- net N$69: now also R421.2; no longer R420.2
- net N$71: now also R420.1; no longer R419.1
- net N$8: now also R316.2; no longer R315.2
- net RA: now also R118.2; no longer R119.2
- net RB: now also R118.1; no longer R119.1
- net SCLK_: now also C105.2, C205.2, C305.2, C406.2; no longer C106.2, C206.2, C306.2, C407.2
- net SOUT101: now also R216.1; no longer R215.1
- net SOUT201: now also R316.1; no longer R315.1
- net SOUT301: now also R416.1; no longer R415.1
- net VCC: now also R115.2, R119.2, R121.1, R215.2, R218.2, R220.1, R315.2, R318.2, R320.1, R415.2, R418.2, R421.1; no longer R101.2, R116.2, R120.1, R201.2, R216.2, R219.1, R301.2, R316.2, R319.1, R401.2, R416.2, R420.1
- net VPRG_: now also R101.1, R201.1, R301.1, R401.1; no longer C102.2, C202.2, C302.2, C402.2, TP16.1, TP29.1, TP39.1, TP8.1
- net XLAT_: now also C102.2, C202.2, C302.2, C402.2; no longer C403.2
Other:
- note added: "09"
- note added: "39,06"
- note added: "Imax"
- note added: "P/ RX=2k4 --> Imax=16,275mA"
- note added: "P/ RX=3k9 --> Imax=10,015mA"
- note added: "RX="
- note added: "The maximum output current per channel"
- note added: "is programmed by a single resistor."
- note removed: "08"
- moved on the sheet: C102, C103, C104, C105, C202, C203, C204, C205, C302, C303, C304, C305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
