File: DIDV_-_Conector_DIDV_BEEB.sch (EAGLE design)
At the start: 6 parts

Commit message: Revisão 9
- Corrigidos algumas falhas de ligação
- Implementação com VPRG dos TLCs via Hardware
- Inserção do cálculo do Riref

Obs. Se somente a criação de boards, não será incrementado. No caso, se criado um board novo board vou subir para 9.1 e assim por diante.
Other:
- note added: "09"
- note added: "Conector parara interligacao entre a placa principal e a expansao."
- note removed: "08"
Changed lines of the file:
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@@
 <text x="203.2" y="29.464" size="1.778" layer="150" font="vector">Dispositivo de Interface para</text>
 <text x="210.82" y="26.162" size="1.778" layer="150" font="vector">Deficientes Visuais</text>
-<text x="250.698" y="10.16" size="2.54" layer="150" font="vector">08</text>
+<text x="250.698" y="10.16" size="2.54" layer="150" font="vector">09</text>
 <text x="7.62" y="7.62" size="6.4516" layer="97" font="vector" ratio="20">Baixa--&gt;Alta</text>
+<text x="7.62" y="17.78" size="2.54" layer="150" font="vector">Conector parara interligacao entre a placa principal e a expansao.</text>
 </plain>
 <instances>
@@
 <text x="203.2" y="29.464" size="1.778" layer="150" font="vector">Dispositivo de Interface para</text>
 <text x="210.82" y="26.162" size="1.778" layer="150" font="vector">Deficientes Visuais</text>
-<text x="250.698" y="10.16" size="2.54" layer="150" font="vector">08</text>
+<text x="250.698" y="10.16" size="2.54" layer="150" font="vector">09</text>
 <text x="7.62" y="7.62" size="6.4516" layer="97" font="vector" ratio="20">Alta--&gt;Baixa</text>
+<text x="7.62" y="15.24" size="2.54" layer="150" font="vector">Conector parara interligacao entre a placa principal e a expansao.</text>
 </plain>
 <instances>

Commit message: Revisão 10
Revisão representa o estado final do projeto, alterações agora somente referentes a valores de componentes e adaptações se e somente se não existir a possibilidade de manobras via software.

Placas nas dimensões e condições as quais foram submetidas a cotação para confecção em local especializado.
Other:
- note added: "10"
- note removed: "09"
Changed lines of the file:
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@@
 <text x="203.2" y="29.464" size="1.778" layer="150" font="vector">Dispositivo de Interface para</text>
 <text x="210.82" y="26.162" size="1.778" layer="150" font="vector">Deficientes Visuais</text>
-<text x="250.698" y="10.16" size="2.54" layer="150" font="vector">09</text>
+<text x="250.698" y="10.16" size="2.54" layer="150" font="vector">10</text>
 <text x="7.62" y="7.62" size="6.4516" layer="97" font="vector" ratio="20">Baixa--&gt;Alta</text>
 <text x="7.62" y="17.78" size="2.54" layer="150" font="vector">Conector parara interligacao entre a placa principal e a expansao.</text>
@@
 <text x="203.2" y="29.464" size="1.778" layer="150" font="vector">Dispositivo de Interface para</text>
 <text x="210.82" y="26.162" size="1.778" layer="150" font="vector">Deficientes Visuais</text>
-<text x="250.698" y="10.16" size="2.54" layer="150" font="vector">09</text>
+<text x="250.698" y="10.16" size="2.54" layer="150" font="vector">10</text>
 <text x="7.62" y="7.62" size="6.4516" layer="97" font="vector" ratio="20">Alta--&gt;Baixa</text>
 <text x="7.62" y="15.24" size="2.54" layer="150" font="vector">Conector parara interligacao entre a placa principal e a expansao.</text>
