File: DIDV_-_Controle_Corrente_Total.sch (EAGLE design)
At the start: 145 parts, among them IC401 PIC18F4550_TQFP44, K401 G5L, Q402 BC817, Q501 FZT493, Q502 FZT493, U201 ACS712LC, U202 ACS712LC, U203 ACS712LC, U301 LM35CAZ, U302 LM35CAZ, U303 LM35CAZ, X101 MINI-USB-32005-301

Commit message: Revisão 10
Revisão representa o estado final do projeto, alterações agora somente referentes a valores de componentes e adaptações se e somente se não existir a possibilidade de manobras via software.

Placas nas dimensões e condições as quais foram submetidas a cotação para confecção em local especializado.
Parts:
- removed C206, C209: (no value), rcl:C-USC0805
- removed C207, C208, C210, C211, C212, C409, C601, C602: 10n, rcl:C-USC0603K
- removed C407: 10nf/50V, rcl:C-EUC0603K
- removed C408: 100n, rcl:C-USC0603
- removed C410, C411, C412, C413, C414: 10n, rcl:C-USC0805K
- removed D403: BAS21, diode:BAS19
- removed D404: BAS70, diode:BAS40
- removed D601, D602: (no value), led:LEDMINI-TOP
- removed F101, F102, F103: 10A/250V, fuse:KS9V
- removed IC401: PIC18F4550_TQFP44, microchip:PIC18F4550_TQFP
- removed JP102, JP103, JP104, JP105, JP106, JP107, JP108, JP109, JP110, JP111, JP112, JP113, JP114, JP115, JP116, JP117, JP118, JP119, JP120, JP121, JP122, JP123, JP124, JP125, JP126, JP127: (no value), jumper:JP1E
- removed K401: G5L, relay:G5L
- removed LED101, LED102, LED103: (no value), led:LED3MM
- removed LOGO201, LOGO301, LOGO401, LOGO501: OSHW-LOGOM, SparkFun-Aesthetics:OSHW-LOGOM
- removed Q401: (no value), crystal:CRYSTALSM49
- removed Q402: BC817, transistor-npn:BC817-16LT1SMD
- removed Q602, Q604: (no value), transistor:BC817-25LT1-NPN-SOT23-BEC
- removed R1, R2: 22R, rcl:R-US_R0603
- removed R408: 100, rcl:R-US_R0603
- removed R409: 1M, rcl:R-US_R0603
- removed R410, R411, R601, R606: 10k, rcl:R-US_R0603
- removed R412, R602, R605: 100k, rcl:R-US_R0603
- removed R413: 1k5, rcl:R-US_R0603
- removed R603, R604: 270, rcl:R-US_R0603
- removed S401: (no value), SparkFun-Electromechanical:TAC_SWITCHPTH
- removed SJ401, SJ402, SJ403, SJ404, SJ405: JUMPER-PAD-3-2OF3_NC_BY_PASTE, SparkFun-Passives:JUMPER-PAD-3-2OF3_NC_BY_PASTE
- removed TP100: USB_In, SparkFun-Passives:TEST-POINT3X4
- removed U201, U202, U203: ACS712LC, allegro-micro:ACS712LC
- removed X101: MINI-USB-32005-301, con-cypressindustries:MINI-USB-32005-301
- added C104, C110, C111, C113, C308, C311: 10n, rcl:C-USC0805K
- added C105: 100n, rcl:C-USC0603
- added C106: 1u, rcl:C-USC0805K
- added C107, C112: 10n, rcl:C-USC0603
- added C108: 10nf/50V, rcl:C-EUC0603K
- added C109, C307, C310, C312: 10n, rcl:C-USC0603K
- added C309: 100nF/50V, rcl:C-USC0805
- added D101: ESDAXXL, diode:ESDAXXL
- added D104: BAS70, diode:BAS40
- added D201, D202: (no value), led:LEDTOPLED-SANTANA
- added F201, F202, F203: 10A/250V, fuse:KS9V
- added IC101: PIC18F4550_TQFP44, microchip:PIC18F4550_TQFP
- added JP201, JP202, JP203, JP204, JP205, JP206, JP207: (no value), jumper:JP1EY
- added K101: G5L, relay:G5L
- added LED201, LED202, LED203: (no value), led:LEDP-LCC-2
- added Q101: (no value), crystal:CRYSTALSM49
- added Q102, Q201, Q202: BC817, transistor-npn:BC817-16LT1SMD
- added R104: 1M, rcl:R-US_R0603
- added R105: 100, rcl:R-US_R0603
- added R106, R107, R403, R406: 10k, rcl:R-US_R0603
- added R108, R404: 100k, rcl:R-US_R0603
- added R109: 1k5, rcl:R-US_R0603
- added R110: 2k, rcl:R-US_R0603
- added R111: 1k3, rcl:R-US_R0603
- added R207: 470, rcl:R-US_R1206
- added R208, R209: 110, rcl:R-US_R1206
- added S101: (no value), SparkFun-Electromechanical:TAC_SWITCHPTH
- added TP1, TP2, TP3, TP4, TP5: TPB1,27, testpad:TPB1,27
- added TP10, TP11: TP-063, keystone_Gordo:TP-063
- added TP12, TP13, TP14, TP15, TP6, TP7, TP8, TP9: TP-063, keystone:TP-063
- added U401, U402, U403: LM35CAZ, NSC_By_element14_Batch_1.1:LM35CAZ
- C101: value 2200uf/35V -> 100n; device rcl:CPOL-EUE3.5-10 -> rcl:C-USC0603
- C102, C103: value 2200uf/35V -> 15p; device rcl:CPOL-EUE3.5-10 -> rcl:C-USC0603K
- C201, C204: value (none) -> 2200uf/35V; device rcl:C-USC0603 -> rcl:CPOL-EUE3.5-10
- C202: value (none) -> 10n
- C203: value (none) -> 2200uf/35V; device rcl:C-USC0805 -> rcl:CPOL-EUE3.5-10
- C205: device rcl:C-USC0603K -> rcl:C-USC0603
- C301, C302, C304: value 10n -> 1nF/50V; device rcl:C-USC0603K -> rcl:C-USC0603
- C303, C305: value 10n -> 100nF/50V; device rcl:C-USC0603K -> rcl:C-USC0805
- C306, C403: device rcl:C-USC0603K -> rcl:C-USC0805K
- C401: value 15p -> 10n; device rcl:C-USC0603K -> rcl:C-USC0805K
- C402: value 15p -> 10n
- C404: value 100n -> 10n; device rcl:C-USC0603 -> rcl:C-USC0603K
- C405: value 1u -> 10n; device rcl:C-USC0603K -> rcl:C-USC0805K
- C406: device rcl:C-USC0805K -> rcl:C-USC0603K
- D102: value ESDAXXL -> BAS21; device diode:ESDAXXL -> diode:BAS19
- JP101: value (none) -> USB_MICROB_PLUGCONN-11752; device jumper:JP1E -> SparkFun-Connectors:USB_MICROB_PLUGCONN-11752
- LOGO101: value OSHW-LOGOM -> OSHW-LOGOL; device SparkFun-Aesthetics:OSHW-LOGOM -> OpenHW_BOT:OSHW-LOGOL
- Q501, Q502: value FZT493 -> BC817; device zetex:FZT493 -> transistor-npn:BC817-16LT1SMD
- R101: value 470 -> 100; device rcl:R-US_0613/5V -> rcl:R-US_R0603
- R102, R103: value 470 -> 22R; device rcl:R-US_0613/5V -> rcl:R-US_R0603
- R201: value 100k -> 470; device rcl:R-US_R0603 -> rcl:R-US_R1206
- R202: value 100k -> 3k
- R203: value 10k -> 2k
- R204: value 100k -> 2k
- R205: value 10k -> 3k
- R206: value 10k -> 470; device rcl:R-US_R0603 -> rcl:R-US_R1206
- R401: value 150k -> 100k
- R405: value 100 -> 10k
- R501, R503: value 150k -> 2k; device rcl:R-US_R1206 -> rcl:R-US_R0603
- R502, R504: value 100k -> 1k3; device rcl:R-US_R1206 -> rcl:R-US_R0603
- U301, U302, U303: value LM35CAZ -> ACS712LC; device NSC_By_element14_Batch_1.1:LM35CAZ -> allegro-micro:ACS712LC
Connections:
- removed net +D: R1.2
- removed net -D: R2.2
- removed net 12V_EN: IC401.RD6/SPP6/P1C
- removed net 6V: U202.IP+, U202.IP+@2
- removed net AGND: C101.-, C102.-, C103.-, C201.2, C202.2, C203.2, C204.2, C206.2, C209.2, C407.2, C501.2, C502.2, IC401.RA1/AN1, IC401.RA4/T0CKI/CIOUT/RCV, IC401.RE1/AN6/CK2SPP, IC401.VSS, IC401.VSS@1, JP102.1, JP102.2, JP103.2, JP104.2, JP108.1, JP108.2, JP109.1, JP109.2, JP110.1, JP110.2, JP111.1, JP112.2, JP113.2, JP116.1, JP116.2, JP117.1, JP117.2, JP118.2, JP119.1, JP120.2, JP124.1, JP124.2, JP125.1, JP125.2, JP126.1, JP126.2, JP127.1, LED101.C, LED102.C, LED103.C, Q402.E, Q501.E, Q502.E, R402.1, R502.1, R504.1, U201.GND, U202.GND, U203.GND
- removed net CTRL_B: IC401.RB3/AN9/CCP2/VPO
- removed net D+_: IC401.RC5/D+/VP, SJ401.2
- removed net D-_: IC401.RC4/D-/VM, SJ403.2
- removed net MCLR_: SJ405.1
- removed net N$20: IC401.RD0/SPP0
- removed net N$25: IC401.RB2/AN8/INT2/VMO
- removed net N$65: R405.2, S401.4
- removed net PGC_OUT: SJ402.3
- removed net PGD_OUT: SJ404.3
- removed net RB6: SJ402.1
- removed net RB7: SJ404.1
- removed net RC4: SJ403.1
- removed net RC5: SJ401.1
- removed net RESET: R413.1, SJ405.3
- removed net _6V: F103.2, U202.IP-, U202.IP-@4
- new net 444: C204.+, F203.2, U302.IP-, U302.IP-@4
- new net GND1: C204.-, LED203.C, TP11.1, TP13.1
- new net N$16: IC101.RD6/SPP6/P1C
- new net N$24: IC101.RB3/AN9/CCP2/VPO
- new net N$45: R101.1, S101.1, S101.2
- new net N$46: F202.1, TP6.1
- new net N$68: IC101.RB2/AN8/INT2/VMO
- net +12V: now also D104.C, D501.C, D502.C, JP204.1, JP205.1, JP206.2, K101C.1, R201.2, U$501.+, U$502.+, U303.IP+, U303.IP+@2; no longer C101.+, JP112.1, JP113.1, JP119.2, R101.2, U203.IP+, U203.IP+@2
- net +6V: now also R207.2, TP12.1, U302.IP+, U302.IP+@2; no longer C103.+, JP118.1, JP120.1, JP127.2, R103.2
- net AN_12V: now also C311.1, R306.2, U303.VIOUT; no longer C211.1, R206.2, U203.VIOUT
- net AN_12V_: now also C312.1, IC101.RA3/AN3/VREF+, R304.1, R306.1; no longer C212.1, IC401.RA3/AN3/VREF+, R204.1, R206.1
- net AN_6V: now also C308.1, R305.2, U302.VIOUT; no longer C208.1, R205.2, U202.VIOUT
- net AN_6V_: now also C310.1, IC101.RA2/AN2/VREF-/CVREF, R302.1, R305.1; no longer C210.1, IC401.RA2/AN2/VREF-/CVREF, R202.1, R205.1
- net AN_VCC: now also C306.1, R303.2, U301.VIOUT; no longer C205.1, R203.2, U201.VIOUT
- net AN_VCC_: now also C307.1, IC101.RA0/AN0, R301.1, R303.1; no longer C207.1, IC401.RA0/AN0, R201.1, R203.1
- net COOLERS: now also IC101.RC2/CCP1/P1A; no longer IC401.RC2/CCP1/P1A
- net D+: now also IC101.RC5/D+/VP, R102.2; no longer SJ401.3
- net D-: now also IC101.RC4/D-/VM, R103.2; no longer SJ403.3
- net GND: now also C101.2, C102.2, C103.2, C104.2, C105.2, C106.2, C107.2, C108.2, C109.2, C110.2, C111.2, C112.2, C113.2, C201.-, C202.2, C203.-, C307.2, C308.2, C309.2, C310.2, C311.2, C312.2, C501.2, C502.2, D101.C2, IC101.RA1/AN1, IC101.RA4/T0CKI/CIOUT/RCV, IC101.RD0/SPP0, IC101.RE1/AN6/CK2SPP, IC101.VSS, IC101.VSS@1, JP101.GND, JP101.SHIELD, JP201.2, JP202.1, JP203.1, JP204.2, JP205.2, JP206.1, JP207.2, LED201.C, LED202.C, Q102.E, Q201.E, Q202.E, Q501.E, Q502.E, R101.2, R108.2, R111.1, R203.2, R401.2, R402.2, R404.2, R502.1, R504.1, TP5.TP, TP7.1, TP9.1, U401.GND, U402.GND, U403.GND; no longer C207.2, C208.2, C210.2, C211.2, C212.2, C408.2, C409.2, C410.2, C411.2, C412.2, C413.2, C414.2, C601.2, C602.2, D102.C2, Q602.E, Q604.E, R201.2, R202.2, R412.2, R602.2, R605.2, S401.2, X101.5
- net MCLR: now also IC101.!MCLR!/VPP/RE3, R109.1, TP2.TP; no longer IC401.!MCLR!/VPP/RE3, SJ405.2
- net N$1: now also LED202.A, R206.1; no longer LED102.A, R102.1
- net N$10: now also D202.A, R209.2; no longer D602.A, R604.2
- net N$11: now also D102.C, R107.2; no longer D403.C, R411.2
- net N$12: now also C301.1, U301.FILTER; no longer C201.1, U201.FILTER
- net N$13: now also C205.1, Q202.B, R202.1, R203.1; no longer C601.1, Q604.B, R601.1, R602.1
- net N$15: now also C202.1, Q201.B, R204.1, R205.2; no longer C602.1, Q602.B, R605.1, R606.2
- net N$17: now also IC101.RB4/AN11/KBI0/CSSPP; no longer IC401.RB4/AN11/KBI0/CSSPP
- net N$18: now also IC101.RB5/KBI1/PGM; no longer IC401.RB5/KBI1/PGM
- net N$19: now also IC101.RC1/T1OSI/ICCP2/!UOE; no longer IC401.RC1/T1OSI/ICCP2/!UOE
- net N$2: now also C302.1, U302.FILTER; no longer C202.1, U202.FILTER
- net N$21: now also Q501.C; no longer Q501.C1, Q501.C2
- net N$22: now also IC101.RC6/TX/CK; no longer IC401.RC6/TX/CK
- net N$23: now also IC101.RC0/TIOSO/T13CKI; no longer IC401.RC0/TIOSO/T13CKI
- net N$26: now also IC101.RD7/SPP7/P1D; no longer IC401.RD7/SPP7/P1D
- net N$28: now also D104.A, K101C.2, Q102.C; no longer D404.A, K401C.2, Q402.C
- net N$29: now also C108.1, Q102.B, R110.1, R111.2; no longer C407.1, Q402.B, R401.1, R402.2
- net N$3: now also C103.1, Q101.2, R105.1; no longer F102.1, JP105.1, JP105.2, JP106.1, JP106.2, JP107.1, JP107.2
- net N$30: now also D201.C, Q202.C; no longer D601.C, Q604.C
- net N$31: now also D202.C, Q201.C; no longer D602.C, Q602.C
- net N$33: now also JP101.D-, R103.1; no longer R2.1, X101.2
- net N$35: now also IC101.NC/ICDT/ICPGD; no longer IC401.NC/ICDT/ICPGD
- net N$36: now also IC101.NC/ICCK/ICPGC; no longer IC401.NC/ICCK/ICPGC
- net N$37: now also D101.C1, JP101.D+, R102.1; no longer D102.C1, R1.1, X101.3
- net N$38: now also IC101.RB1/AN10/INT1/SCK/SCL; no longer IC401.RB1/AN10/INT1/SCK/SCL
- net N$39: now also IC101.RB0/AN12/INT0/LFT0/SDI/SDA; no longer IC401.RB0/AN12/INT0/LFT0/SDI/SDA
- net N$4: now also LED201.A, R201.1; no longer LED101.A, R101.1
- net N$40: now also IC101.RD5/SPP5/P1B; no longer IC401.RD5/SPP5/P1B
- net N$41: now also IC101.RC7/RX/DT/SDO; no longer IC401.RC7/RX/DT/SDO
- net N$43: now also IC101.NC/ICPORTS; no longer IC401.NC/ICPORTS
- net N$44: now also IC101.NC/!ICRST!/IVVPP; no longer IC401.NC/!ICRST!/IVVPP
- net N$5: now also F201.1, TP8.1; no longer F101.1, JP101.1, JP101.2, JP114.1, JP114.2, JP115.1, JP115.2
- net N$6: now also C304.1, U303.FILTER; no longer C204.1, U203.FILTER
- net N$7: now also LED203.A, R207.1; no longer LED103.A, R103.1
- net N$71: now also Q502.C; no longer Q502.C1, Q502.C2
- net N$8: now also F203.1, TP10.1; no longer F103.1, JP121.1, JP121.2, JP122.1, JP122.2, JP123.1, JP123.2
- net N$9: now also D201.A, R208.1; no longer D601.A, R603.1
- net OSC1: now also C102.1, IC101.OSC1/CLKI, Q101.1, R104.1; no longer C401.1, IC401.OSC1/CLKI, Q401.1, R408.1, R408.2, R409.1
- net OSC2: now also IC101.RA6/OSC2/CLKO, R104.2, R105.2; no longer C402.1, IC401.RA6/OSC2/CLKO, Q401.2, R409.2
- net PGC: now also IC101.RB6/KBI2/PGC, TP1.TP; no longer IC401.RB6/KBI2/PGC, SJ402.2
- net PGD: now also IC101.RB7/BKI3/PGD, TP3.TP; no longer IC401.RB7/BKI3/PGD, SJ404.2
- net SD: now also IC101.RD4/SPP4, R110.2; no longer IC401.RD4/SPP4, R401.2
- net TS1: now also C401.1, R403.2, U401.VOUT; no longer C301.1, R303.2, U301.VOUT
- net TS1_: now also C402.1, IC101.RA5/AN4/!SS!/HLVDIN/C2OUT, R401.1, R403.1; no longer C302.1, IC401.RA5/AN4/!SS!/HLVDIN/C2OUT, R301.1, R303.1
- net TS2: now also C403.1, R405.2, U402.VOUT; no longer C303.1, R305.2, U302.VOUT
- net TS2_: now also C404.1, IC101.RE0/AN5/CK1SPP, R402.1, R405.1; no longer C304.1, IC401.RE0/AN5/CK1SPP, R302.1, R305.1
- net TS3: now also C405.1, R406.2, U403.VOUT; no longer C305.1, R306.2, U303.VOUT
- net TS3_: now also C406.1, IC101.RE2/AN7/OESPP, R404.1, R406.1; no longer C306.1, IC401.RE2/AN7/OESPP, R304.1, R306.1
- net USBCON: now also IC101.RD3/SPP3, R205.1; no longer IC401.RD3/SPP3, R601.2
- net USBTXRX: now also IC101.RD2/SPP2, R202.2; no longer IC401.RD2/SPP2, R606.1
- net USB_IN: now also C109.1, IC101.RD1/SPP1, R106.1, R108.1; no longer C409.1, IC401.RD1/SPP1, R410.1, R412.1, TP100.1
- net U_MCLR: now also C106.1, R107.1, R109.2, S101.3, S101.4; no longer C405.1, R405.1, R411.1, R413.2
- net VCC: now also C107.1, C110.1, C111.1, C112.1, C113.1, C303.1, C305.1, C309.1, D102.A, IC101.VDD, IC101.VDD@1, JP201.1, JP202.2, JP203.2, JP207.1, R206.2, R208.2, R209.1, TP4.TP, U301.IP+, U301.IP+@2, U301.VCC, U302.VCC, U303.VCC, U401.+VS, U402.+VS, U403.+VS; no longer C102.+, C203.1, C206.1, C209.1, C406.1, C410.1, C411.1, C412.1, C413.1, C414.1, D403.A, D404.C, D501.C, D502.C, IC401.VDD, IC401.VDD@1, JP103.1, JP104.1, JP111.2, K401C.1, R102.2, R603.2, R604.1, U$501.+, U$502.+, U201.IP+, U201.IP+@2, U201.VCC, U202.VCC, U203.VCC, U301.+VS, U302.+VS, U303.+VS
- net VUSB: now also C104.1, JP101.VCC, R106.2; no longer C403.1, R410.2, X101.1
- net VUSB_: now also C101.1, C105.1, IC101.VUSB; no longer C404.1, C408.1, IC401.VUSB
- net WG1: now also K101-A.COM, TP15.1; no longer K401-A.COM
- net WG2: now also K101-A.NC, TP14.1; no longer K401-A.NC
- net _+12V: now also C201.+, F201.2, U303.IP-, U303.IP-@4; no longer F101.2, U203.IP-, U203.IP-@4
- net _VCC: now also C203.+, F202.2, U301.IP-, U301.IP-@4; no longer F102.2, U201.IP-, U201.IP-@4
Other:
- note added: "10"
- note added: "Hall_Current_6V"
- note added: "OM"
- note added: "Test points para gravação"
- note removed: "09"
- note removed: "Funcao"
- note removed: "Hall_Current_3V3"
- note removed: "Seletores"
